File: Lab 1/Lab 1.kicad_sch (KiCad schematic)
At the start: 62 parts, among them K1 Fujitsu_FTR-LYCA005x, K10 Fujitsu_FTR-LYCA005x, K11 Fujitsu_FTR-LYCA005x, K12 Fujitsu_FTR-LYCA005x, K2 Fujitsu_FTR-LYCA005x, K3 Fujitsu_FTR-LYCA005x, K4 Fujitsu_FTR-LYCA005x, K5 Fujitsu_FTR-LYCA005x, K6 Fujitsu_FTR-LYCA005x, K7 Fujitsu_FTR-LYCA005x, K8 Fujitsu_FTR-LYCA005x, K9 Fujitsu_FTR-LYCA005x, M2 Motor_DC, M3 Motor_DC, M4 Motor_DC, SW1 SW_Push, SW10 SW_SPDT_XKB_DMx-xxxx-1, SW11 START, SW12 STOP, SW13 SW_SPDT_XKB_DMx-xxxx-1, SW14 SW_SPDT_XKB_DMx-xxxx-1, SW15 STOP, SW18 START, SW2 SW_Push_Open, SW3 SW_Push, SW4 SW_Push_Open, SW5 SW_Push, SW6 SW_Push, SW7 SW_Push, SW8 SW_Push, SW9 SW_SPDT_XKB_DMx-xxxx-1

Commit message: Redo B2
Parts:
- removed D6, D7, D8, D9: LED, symbol Device:LED
- removed F5: Fuse, symbol Device:Fuse
- removed K4, K7, K8: Fujitsu_FTR-LYCA005x, Relay_THT:Relay_SPDT_Fujitsu_FTR-LYCA005x_FormC_Vertical, symbol Relay:Fujitsu_FTR-LYCA005x
- removed M3: Motor_DC, symbol Motor:Motor_DC
- removed R7: R, symbol Device:R
- removed SW10, SW9: SW_SPDT_XKB_DMx-xxxx-1, symbol Switch:SW_SPDT_XKB_DMx-xxxx-1
- removed SW11: START, symbol Switch:SW_Push
- removed SW12: STOP, symbol Switch:SW_Push_Open
- removed SW7, SW8: SW_Push, symbol Switch:SW_Push
- removed V6: 24 V, symbol Simulation_SPICE:VDC
- removed e5: ~, symbol relay_contact:Thermal_Contact_NC
- added C1, C2, d1: ~, symbol relay_coil:Relay_coil
- added C1 (x2), C2 (x2), d1: ~, symbol relay_contact:Relay_contact
- added F7: Fuse, symbol Device:Fuse
- added L3, L4, L5, L6: ~, symbol Indicator:Indicator
- added M5: Motor_DC, symbol Motor:Motor_DC
- added SW16: START, symbol Switch:SW_Push
- added SW17: STOP, symbol Switch:SW_Push_Open
- added SW19, SW21: SW_Push, symbol Switch:SW_Push
- added SW20, SW22: SW_SPDT_XKB_DMx-xxxx-1, symbol Switch:SW_SPDT_XKB_DMx-xxxx-1
- added e6, e7: ~, symbol relay_contact:Thermal_Contact_NC
Connections:
- net GND: now also K10.A2, K11.12, K9.12
- net at K10.14, K11.14, K11.A1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: now also K10.A1, SW16.2; no longer SW18.2
- net at V7.1: now also F6.1
- net at SW15.2 (B): now also K10.11, SW16.1; no longer K10.A2
- net at K9.11, M4.1 (+): now also D13.2 (A)
- net at D10.2 (A): now also K11.11, M4.2 (-); no longer K9.12
- net at F6.2: no longer SW15.1 (A)
- new net: SW20.1 (A), SW22.1 (A)
- new net: SW17.1 (A), SW18.2
- new net: SW18.1, SW19.2, SW21.2
Other:
- note added: "N"
- note added: "R"
- moved on the sheet: D10, D13, F6

Commit message: Redo B3
Parts:
- removed D10, D11, D12, D13: LED, symbol Device:LED
- removed F6: Fuse, symbol Device:Fuse
- removed K10, K11, K12, K9: Fujitsu_FTR-LYCA005x, Relay_THT:Relay_SPDT_Fujitsu_FTR-LYCA005x_FormC_Vertical, symbol Relay:Fujitsu_FTR-LYCA005x
- removed M4: Motor_DC, symbol Motor:Motor_DC
- removed SW13, SW14: SW_SPDT_XKB_DMx-xxxx-1, symbol Switch:SW_SPDT_XKB_DMx-xxxx-1
- removed SW15: STOP, symbol Switch:SW_Push_Open
- removed SW16: START, symbol Switch:SW_Push
- removed V7: 24 V, symbol Simulation_SPICE:VDC
- removed e6: ~, symbol relay_contact:Thermal_Contact_NC
- added C3, C4, C5, d6: ~, symbol relay_coil:Relay_coil
- added C3 (x2), C4 (x2), C5 (x2), C6, d6: ~, symbol relay_contact:Relay_contact
- added F8: Fuse, symbol Device:Fuse
- added L10, L11, L12, L9: ~, symbol Indicator:Indicator
- added M6: Motor_DC, symbol Motor:Motor_DC
- added SW23: STOP, symbol Switch:SW_Push_Open
- added SW24: START, symbol Switch:SW_Push
- added SW26, SW27: SW_SPDT_XKB_DMx-xxxx-1, symbol Switch:SW_SPDT_XKB_DMx-xxxx-1
- added e8: ~, symbol relay_contact:Thermal_Contact_NC
Connections:
- new net: SW26.2 (B), SW26.3 (C), SW27.1 (A)
- new net: SW23.1 (A), SW24.2
- new net: SW24.1, SW26.1 (A)
- no-connect marks 0 -> 2
